File: udb-s.kicad_pcb (KiCad board)
At the start: 4 copper layers, 40 x 9 mm, 11 parts, among them J1 TYPE-C-31-M-12, J2 78171-0004, U1 TPD4E05U06DQAR

Commit message: Fix Link
Other:
- board text added: "Unified-S1 V1.1 unified- daughterboard.github.io"
- board text removed: "Unified-S1 V1.1 www.unified- daughterboard.github.io"
Changed lines of the file:
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@@
   (gr_line (start 147 90.5) (end 116 90.499999) (layer "Edge.Cuts") (width 0.1))
   (gr_line (start 116 99.500001) (end 147 99.5) (layer "Edge.Cuts") (width 0.1))
-  (gr_text "Unified-S1 V1.1\nwww.unified-\ndaughterboard.github.io" (at 126.25 95) (layer "B.SilkS")
+  (gr_text "Unified-S1 V1.1\nunified-\ndaughterboard.github.io" (at 126.25 95) (layer "B.SilkS")
     (effects (font (size 0.8 0.8) (thickness 0.2)) (justify mirror))
   )
